Commit message: Add files via upload
Mostly fixed launch files except gazebo

File: khi_ux150_description/urdf/khi_ux150_macro.xacro (robot description, xacro)
@@ -198,5 +198,5 @@
     <child link="${prefix}parallel_1"/>
     <axis xyz="0.0 -1.0 0.0"/>
-    <limit lower="-1.13446" upper="1.22173" effort="1000" velocity="1"/>
+    <limit lower="-1.22173" upper="1.13446" effort="1000" velocity="1"/>
 </joint>
 <joint name="${prefix}jt2_1" type="revolute">
